File: pcb.kicad_sch (KiCad schematic)
At the start: 4 parts, among them U1 LTC3240EDC-3_3

Commit message: add header
Parts:
- added J1: Conn_01x03, Connector_PinHeader_2.54mm:PinHeader_1x03_P2.54mm_Vertical, symbol Connector_Generic:Conn_01x03
Connections:
- net +3V3: now also J1.3 (Pin_3)
- net GND: now also J1.2 (Pin_2)
- net VDD: now also J1.1 (Pin_1)
Changed lines of the file:
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@@
+    (stroke (width 0) (type default))
+  )
+  (wire (pts (xy 86.36 88.9) (xy 91.44 88.9))
     (stroke (width 0) (type default))
   )
@@
   )
   (wire (pts (xy 133.35 46.99) (xy 139.7 46.99))
+    (stroke (width 0) (type default))
+  )
+  (wire (pts (xy 86.36 86.36) (xy 91.44 86.36))
+    (stroke (width 0) (type default))
+  )
+  (wire (pts (xy 86.36 91.44) (xy 91.44 91.44))
     (stroke (width 0) (type default))
   )
@@
     )
   )
+  (symbol (lib_id "power:+3V3") (at 86.36 91.44 90) (unit 1)
+    (in_bom yes) (on_board yes) (dnp no) (fields_autoplaced)
+    (property "Reference" "#PWR010" (at 90.17 91.44 0)
+      (effects (font (size 1.27 1.27)) hide)
+    )
+    (property "Value" "+3V3" (at 82.55 91.44 90)
+      (effects (font (size 1.27 1.27)) (justify left))
+    )
+    (property "Footprint" "" (at 86.36 91.44 0)
+      (effects (font (size 1.27 1.27)) hide)
+    )
+    (property "Datasheet" "" (at 86.36 91.44 0)
+      (effects (font (size 1.27 1.27)) hide)
+    )
+    (pin "1")
+    (instances
+      (project "pcb"
+        (path "/8d092590-a518-48e5-bcb8-8b85efb8e7ef"
+          (reference "#PWR010") (unit 1)
+        )
+      )
+      (project "pcb"
+        (path "/c5153b1f-707a-4455-a5f6-332464ea0712"
+          (reference "#PWR01") (unit 1)
+        )
+      )
+    )
+  )
+  (symbol (lib_id "power:VDD") (at 86.36 86.36 90) (unit 1)
+    (in_bom yes) (on_board yes) (dnp no) (fields_autoplaced)
+    (property "Reference" "#PWR09" (at 90.17 86.36 0)
+      (effects (font (size 1.27 1.27)) hide)
+    )
+    (property "Value" "VDD" (at 82.55 86.36 90)
+      (effects (font (size 1.27 1.27)) (justify left))
+    )
+    (property "Footprint" "" (at 86.36 86.36 0)
+      (effects (font (size 1.27 1.27)) hide)
+    )
+    (property "Datasheet" "" (at 86.36 86.36 0)
+      (effects (font (size 1.27 1.27)) hide)
+    )
+    (pin "1")
+    (instances
+      (project "pcb"
+        (path "/8d092590-a518-48e5-bcb8-8b85efb8e7ef"
+          (reference "#PWR09") (unit 1)
+        )
+      )
+    )
+  )
   (symbol (lib_id "power:VDD") (at 144.78 44.45 270) (unit 1)
     (in_bom yes) (on_board yes) (dnp no) (fields_autoplaced)
@@
     )
   )
+  (symbol (lib_id "power:GND") (at 86.36 88.9 270) (unit 1)
+    (in_bom yes) (on_board yes) (dnp no) (fields_autoplaced)
+    (property "Reference" "#PWR08" (at 80.01 88.9 0)
+      (effects (font (size 1.27 1.27)) hide)
+    )
+    (property "Value" "GND" (at 82.55 88.9 90)
+      (effects (font (size 1.27 1.27)) (justify right))
+    )
+    (property "Footprint" "" (at 86.36 88.9 0)
+      (effects (font (size 1.27 1.27)) hide)
+    )
+    (property "Datasheet" "" (at 86.36 88.9 0)
+      (effects (font (size 1.27 1.27)) hide)
+    )
+    (pin "1")
+    (instances
+      (project "pcb"
+        (path "/8d092590-a518-48e5-bcb8-8b85efb8e7ef"
+          (reference "#PWR08") (unit 1)
+        )
+      )
+      (project "pcb"
+        (path "/c5153b1f-707a-4455-a5f6-332464ea0712"
+          (reference "#PWR06") (unit 1)
+        )
+      )
+    )
+  )
   (symbol (lib_id "Device:C_Small") (at 46.99 48.26 0) (unit 1)
     (in_bom yes) (on_board yes) (dnp no) (fields_autoplaced)
@@
         )
       )
+    )
+  )
+  (symbol (lib_id "Connector_Generic:Conn_01x03") (at 96.52 88.9 0) (unit 1)
+    (in_bom yes) (on_board yes) (dnp no) (fields_autoplaced)
+    (property "Reference" "J1" (at 99.06 87.63 0)
+      (effects (font (size 1.27 1.27)) (justify left))
+    )
+    (property "Value" "Conn_01x03" (at 99.06 90.17 0)
+      (effects (font (size 1.27 1.27)) (justify left))
+    )
+    (property "Footprint" "Connector_PinHeader_2.54mm:PinHeader_1x03_P2.54mm_Vertical" (at 96.52 88.9 0)
+      (effects (font (size 1.27 1.27)) hide)
+    )
+    (property "Datasheet" "~" (at 96.52 88.9 0)
+      (effects (font (size 1.27 1.27)) hide)
+    )
+    (pin "1")
+    (pin "2")
+    (pin "3")
+    (instances
+      (project "pcb"
+        (path "/8d092590-a518-48e5-bcb8-8b85efb8e7ef"
+          (reference "J1") (unit 1)
+        )
+      )
