File: pcb.kicad_pcb (KiCad board)
At the start: 2 copper layers, 5 parts, among them J1 Conn_01x03, U1 LTC3240EDC-3_3

Commit message: add pcb wiring
Routing:
- net GND: track 0.00 -> 2.98 mm, vias 0 -> 4
- added copper zone on B.Cu, net GND
- added copper zone on F.Cu, net GND
Other:
- board outline added: 10.2 x 9.1 mm
Changed lines of the file:
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@@
     (property "ki_keywords" "connector")
     (attr through_hole)
-    (fp_text reference "J1" (at 0 -2.33) (layer "F.SilkS")
+    (fp_text reference "J1" (at 1.27 -1.36) (layer "F.SilkS") hide
         (effects (font (size 1 1) (thickness 0.15)))
     )
@@
     )
   )
+  (gr_line (start 68.58 79.756) (end 68.58 70.612)
+    (stroke (width 0.1) (type default)) (layer "Edge.Cuts"))
+  (gr_line (start 58.42 70.612) (end 68.58 70.612)
+    (stroke (width 0.1) (type default)) (layer "Edge.Cuts"))
+  (gr_line (start 58.42 79.756) (end 68.58 79.756)
+    (stroke (width 0.1) (type default)) (layer "Edge.Cuts"))
+  (gr_line (start 58.42 79.756) (end 58.42 70.612)
+    (stroke (width 0.1) (type default)) (layer "Edge.Cuts"))
   (segment (start 67.043 72.631) (end 63.246 72.631) (width 0.2) (layer "F.Cu") (net 1))
   (segment (start 67.455 74.531) (end 67.564 74.422) (width 0.2) (layer "F.Cu") (net 1))
@@
   (segment (start 62.23 74.676) (end 62.23 72.644) (width 0.2) (layer "F.Cu") (net 1))
   (segment (start 66.802 74.531) (end 67.455 74.531) (width 0.2) (layer "F.Cu") (net 1))
+  (segment (start 63.246 74.181) (end 64.602 74.181) (width 0.2) (layer "F.Cu") (net 2))
+  (segment (start 65.377 74.531) (end 65.877 75.031) (width 0.2) (layer "F.Cu") (net 2))
+  (segment (start 64.602 74.181) (end 64.952 74.531) (width 0.2) (layer "F.Cu") (net 2))
+  (segment (start 64.952 74.531) (end 65.377 74.531) (width 0.2) (layer "F.Cu") (net 2))
+  (via (at 64.616174 73.517088) (size 0.8) (drill 0.4) (layers "F.Cu" "B.Cu") (free) (net 2))
+  (via (at 61.976 76.708) (size 0.8) (drill 0.4) (layers "F.Cu" "B.Cu") (free) (net 2))
+  (via (at 67.903147 71.563958) (size 0.8) (drill 0.4) (layers "F.Cu" "B.Cu") (free) (net 2))
+  (via (at 67.68084 78.990084) (size 0.8) (drill 0.4) (layers "F.Cu" "B.Cu") (free) (net 2))
   (segment (start 64.952 75.531) (end 64.952 76.214314) (width 0.2) (layer "F.Cu") (net 3))
   (segment (start 64.262 76.904314) (end 64.262 77.724) (width 0.2) (layer "F.Cu") (net 3))
@@
   (segment (start 66.802 75.531) (end 67.403 75.531) (width 0.2) (layer "F.Cu") (net 5))
   (segment (start 67.564 75.692) (end 67.564 76.2) (width 0.2) (layer "F.Cu") (net 5))
+  (zone (net 2) (net_name "GND") (layers "F&B.Cu") (hatch edge 0.5)
+    (connect_pads (clearance 0.5))
+    (min_thickness 0.25) (filled_areas_thickness no)
+    (fill yes (thermal_gap 0.5) (thermal_bridge_width 0.5))
+    (polygon
+      (pts
+        (xy 69.088 70.104)
+        (xy 69.088 80.264)
+        (xy 57.912 80.264)
+        (xy 57.912 70.104)
+      )
+    )
+  )
 )

Commit message: add pcb text
Other:
- board text added: "1.8v<IN<2.5v-40mA 2.5v<IN<5.5v-150mA"
- board text added: "IN-1.8_5.5V OUT-3.3v"
Changed lines of the file:
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@@
   (gr_line (start 58.42 79.756) (end 58.42 70.612)
     (stroke (width 0.1) (type default)) (layer "Edge.Cuts"))
+  (gr_text "IN-1.8_5.5V\nOUT-3.3v\n" (at 64.008 75.184 90) (layer "B.SilkS")
+    (effects (font (size 0.8 0.8) (thickness 0.2) bold) (justify bottom mirror))
+  )
+  (gr_text "1.8v<IN<2.5v-40mA\n2.5v<IN<5.5v-150mA" (at 67.056 75.184 90) (layer "B.SilkS")
+    (effects (font (size 0.5 0.5) (thickness 0.125)) (justify bottom mirror))
+  )
   (segment (start 67.043 72.631) (end 63.246 72.631) (width 0.2) (layer "F.Cu") (net 1))
   (segment (start 67.455 74.531) (end 67.564 74.422) (width 0.2) (layer "F.Cu") (net 1))
